File: magnos-plasma.kicad_sch (KiCad schematic)
At the start: 64 parts, among them J1 Input, J101 External 5 V / 1 A ceiling, J102 Shield temperature sensor, J103 Propulsor temperature sensor, J104 Frame bond, J105 Service monitor, J201 SH two-pin coil connector, J3 AC Output, J301 PR two-pin coil connector, J4 DC Payload, J401 Two-pin HV feedthrough, J501 Two-pin HV feedthrough, Q2 Darlington NPN, Q5 Darlington NPN, Q8 Darlington NPN, T1 Transformer_1P_2S, T2 Transformer_1P_2S, U1 HHG1D-1, U101 Sequencer / shutdown controll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, U201 Isolated driver / limiter - T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, U301 Isolated driver / limiter - T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, U401 Isolated driver / limiter - T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, U501 Isolated driver / limiter - T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, U601 Gas valve driver + flyback / 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, U602 Isolated neutralizer supply /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, Y2 2500Hz, Y3 Squared 60Hz, Y4 Squared 200KHz, Y5 Squared 250Hz, Y601 Injection valve - rating TBD

Commit message: Begin fix interface
Other:
- note added: "Magnos J3 AC output is wired to the HV rectifier; J4 DC output is wired to the coil drivers."
- moved on the sheet: L201, L301, Z401, Z501

Commit message: Begin fix wiring
Parts:
- added H101: Engine chassis bond, symbol MagnosSystem:H101
- added J601: Valve feedthrough, symbol MagnosSystem:J601
- added J602: Neutralizer feedthrough, symbol MagnosSystem:J602
- added T102: Shield sensor, symbol MagnosSystem:T102
- added T103: Engine sensor, symbol MagnosSystem:T103
- added U701: Magnos isolated booster 1/1; target 1e+07 V / TBD, symbol MagnosSystem:U701
Connections:
- net CHASSIS: now also H101.1, H101.2
- net ENABLE: now also U701.3 (ENABLE)
- net GAS_N: now also J601.2 (RETURN)
- net GAS_P: now also J601.1 (POS)
- net HV_BUS_P: now also U701.5 (OUT+); no longer F102.2
- net HV_RETURN: now also U701.2 (IN-); no longer C101.2, R102.2, TP101.2 (IN-), U401.2 (IN-), U501.2 (IN-), U602.2 (IN-)
- net INPUT_5V: now also T102.1 (VCC), T103.1 (VCC)
- net INPUT_RETURN: now also T102.2 (RETURN), T103.2 (RETURN), U701.4 (CTRL_RTN)
- net NEUT_N: now also J602.2 (RETURN)
- net NEUT_P: now also J602.1 (POS)
- net PR_TEMP: now also T103.3 (SIGNAL)
- net SH_TEMP: now also T102.3 (SIGNAL)
- new net HV_PREBOOST_P: F102.2, U701.1 (IN+)
- new net HV_STACK_RETURN: C101.2, R102.2, TP101.2 (IN-), U401.2 (IN-), U501.2 (IN-), U602.2 (IN-), U701.6 (OUT-)
Other:
- note added: "CASCADED MAGNOS: 1 stage(s), 1e+07 V target. 5 W source; 80% assumed per stage; no power multiplication."

Commit message: Transfer wiring
Other:
- note added: "1 cascaded booster(s); 10 MV target; 5 W input shared, assumed losses. Functional architecture, ratings TBD."
- note added: "MAGNOS PLASMA / ALL CONNECTIONS DRAWN / CROSSINGS CONNECT ONLY AT JUNCTION DOTS"
- note added: "Original beta circuit at left. Three functional columns; named backplane conductors below."
- note removed: "5 V / 1 A source annotation. No verified transformer gain. No TW supply is created by this adapter."
- note removed: "Added interconnect is drawn copper on the 1.27 mm grid. TBD means not specified by the source."
- note removed: "All converter control ports below are isolated functional interfaces. HV return is NOT chassis."
- note removed: "CASCADED MAGNOS: 1 stage(s), 1e+07 V target. 5 W source; 80% assumed per stage; no power multiplication."
- note removed: "HV electrode branches + coil channels + valve + neutralizer SHARE the available input power."
- note removed: "MAGNOS PLASMA SYSTEM - COMPLETE FUNCTIONAL WIRING / UNVALIDATED HARDWARE"
- note removed: "Magnos J3 AC output is wired to the HV rectifier; J4 DC output is wired to the coil drivers."
- note removed: "Original beta circuit retained at left. Added blocks require circuit design and rated parts before construction."
- note removed: "TBD means not specified by source. This is a wired functional architecture, not a fabrication-ready design."
- moved on the sheet: J101, J102, J103, J104, J105, J201, J301, J401, J501, J601, J602, L201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
